Commit message: Initialize base properties, footprint and base links

File: robot_description/urdf/mobile_base.xacro (robot description, xacro)
@@ -1,3 +1,21 @@
 <? xml version="1.0"?>
 <robot xmlns:xacro="http://www.ros.org/wiki/xacro">
+<!-- Define mobile base properties -->
+<property name="base_length" value="0.6"/>
+<property name="base_width" value="0.4"/>
+<property name="base_height" value="0.2"/>
+<property name="wheel_radius" value="0.1"/>
+<property name="wheel_width" value="0.05"/>
+<!-- Base footprint -->
+<link name="base_footprint"/>
+<!--Mobile base link-->
+<link name="mobile_base">
+    <visual>
+        <geometry>
+            <box size="${base_length} ${base_width} ${base_height}"/>
+        </geometry>
+        <origin xyz="0 0 0" rpy="0 0 0"/>
+        <material name="blue"/>
+    </visual>
+</link>
 </robot>

Commit message: Initialize links with basics

File: robot_description/urdf/mobile_base.xacro (robot description, xacro)
@@ -7,4 +7,5 @@
 <property name="wheel_radius" value="0.1"/>
 <property name="wheel_width" value="0.05"/>
+<property name="caster_radius" value="0.05"/>
 <!-- Base footprint -->
 <link name="base_footprint"/>
@@ -19,3 +20,28 @@
     </visual>
 </link>
+<!-- Wheels links -->
+<xacro:macro name="wheel_link" params="prefix">
+    <link name="${prefix}_wheel">
+        <visual>
+            <geometry>
+                <cylinder radius="${wheel_radius}" length="${wheel_width}"/>
+            </geometry>
+            <origin xyz="0 0 0" rpy="0 0 0"/>
+            <material name="grey"/>
+        </visual>
+    </link>
+</xacro:macro>
+<!-- Instantiate wheel links -->
+<xacro:wheel_link prefix="left_wheel"/>
+<xacro:wheel_link prefix="right_wheel"/>
+<!-- Caster wheel link -->
+<link name="caster_wheel">
+    <visual>
+        <geometry>
+            <sphere radius="${caster_radius}"/>
+        </geometry>
+        <origin xyz="0 0 0" rpy="0 0 0"/>
+        <material name="grey"/>
+    </visual>
+</link>
 </robot>

Commit message: Initialize joints with basics

File: robot_description/urdf/mobile_base.xacro (robot description, xacro)
@@ -8,8 +8,7 @@
 <property name="wheel_width" value="0.05"/>
 <property name="caster_radius" value="0.05"/>
-<!-- Base footprint -->
+<!-- Links -->
 <link name="base_footprint"/>
-<!--Mobile base link-->
-<link name="mobile_base">
+<link name="mobile_base_link">
     <visual>
         <geometry>
@@ -20,7 +19,6 @@
     </visual>
 </link>
-<!-- Wheels links -->
 <xacro:macro name="wheel_link" params="prefix">
-    <link name="${prefix}_wheel">
+    <link name="${prefix}_wheel_link">
         <visual>
             <geometry>
@@ -32,9 +30,7 @@
     </link>
 </xacro:macro>
-<!-- Instantiate wheel links -->
 <xacro:wheel_link prefix="left_wheel"/>
 <xacro:wheel_link prefix="right_wheel"/>
-<!-- Caster wheel link -->
-<link name="caster_wheel">
+<link name="caster_wheel_link">
     <visual>
         <geometry>
@@ -45,3 +41,24 @@
     </visual>
 </link>
+<!-- Joints -->
+<joint name="base_joint" type="fixed">
+    <parent link="base_footprint"/>
+    <child link="mobile_base_link"/>
+    <origin xyz="0 0 0" rpy="0 0 0"/>
+</joint>
+<joint name="left_wheel_joint" type="continuous">
+    <parent link="mobile_base_link"/>
+    <child link="left_wheel_link"/>
+    <origin xyz="0 0 0" rpy="0 0 0"/>
+</joint>
+<joint name="right_wheel_joint" type="continuous">
+    <parent link="mobile_base_link"/>
+    <child link="right_wheel_link"/>
+    <origin xyz="0 0 0" rpy="0 0 0"/>
+</joint>
+<joint name="caster_wheel_joint" type="fixed">
+    <parent link="mobile_base_link"/>
+    <child link="caster_wheel_link"/>
+    <origin xyz="0 0 0" rpy="0 0 0"/>
+</joint>
 </robot>

Commit message: updated code for axis

File: robot_description/urdf/mobile_base.xacro (robot description, xacro)
@@ -51,4 +51,5 @@
     <child link="left_wheel_link"/>
     <origin xyz="0 0 0" rpy="0 0 0"/>
+    <axis xyz="0 1 0"/>
 </joint>
 <joint name="right_wheel_joint" type="continuous">
@@ -56,4 +57,5 @@
     <child link="right_wheel_link"/>
     <origin xyz="0 0 0" rpy="0 0 0"/>
+    <axis xyz="0 1 0"/>
 </joint>
 <joint name="caster_wheel_joint" type="fixed">

Commit message: fixed typo

File: robot_description/urdf/mobile_base.xacro (robot description, xacro)
@@ -2,10 +2,10 @@
 <robot xmlns:xacro="http://www.ros.org/wiki/xacro">
 <!-- Define mobile base properties -->
-<property name="base_length" value="0.6"/>
-<property name="base_width" value="0.4"/>
-<property name="base_height" value="0.2"/>
-<property name="wheel_radius" value="0.1"/>
-<property name="wheel_width" value="0.05"/>
-<property name="caster_radius" value="0.05"/>
+<xacro:property name="base_length" value="0.6"/>
+<xacro:property name="base_width" value="0.4"/>
+<xacro:property name="base_height" value="0.2"/>
+<xacro:property name="wheel_radius" value="0.1"/>
+<xacro:property name="wheel_width" value="0.05"/>
+<xacro:property name="caster_radius" value="0.05"/>
 <!-- Links -->
 <link name="base_footprint"/>

Commit message: modified joint and links orientations

File: robot_description/urdf/mobile_base.xacro (robot description, xacro)
@@ -25,5 +25,5 @@
                 <cylinder radius="${wheel_radius}" length="${wheel_width}"/>
             </geometry>
-            <origin xyz="0 0 0" rpy="0 0 0"/>
+            <origin xyz="0 0 0" rpy="0 ${pi/2} ${-pi/2}"/>
             <material name="grey"/>
         </visual>
@@ -45,10 +45,10 @@
     <parent link="base_footprint"/>
     <child link="mobile_base_link"/>
-    <origin xyz="0 0 0" rpy="0 0 0"/>
+    <origin xyz="0 0 ${wheel_radius + base_height/2}" rpy="0 0 0"/>
 </joint>
 <joint name="left_wheel_joint" type="continuous">
     <parent link="mobile_base_link"/>
     <child link="left_wheel_link"/>
-    <origin xyz="0 0 0" rpy="0 0 0"/>
+    <origin xyz="${-base_length/4} ${-(base_width + wheel_width)/2} ${-(base_height/2)}" rpy="0 0 0"/>
     <axis xyz="0 1 0"/>
 </joint>
@@ -56,5 +56,5 @@
     <parent link="mobile_base_link"/>
     <child link="right_wheel_link"/>
-    <origin xyz="0 0 0" rpy="0 0 0"/>
+    <origin xyz="${-base_length/4} ${(base_width + wheel_width)/2} ${-(base_height/2)}" rpy="0 0 0"/>
     <axis xyz="0 1 0"/>
 </joint>
@@ -62,5 +62,5 @@
     <parent link="mobile_base_link"/>
     <child link="caster_wheel_link"/>
-    <origin xyz="0 0 0" rpy="0 0 0"/>
+    <origin xyz="${base_length/4} 0 ${-(caster_radius+base_height/2)}" rpy="0 0 0"/>
 </joint>
 </robot>

Commit message: Add collision and inertia

File: robot_description/urdf/mobile_base.xacro (robot description, xacro)
@@ -18,4 +18,11 @@
         <material name="blue"/>
     </visual>
+    <collision>
+        <geometry>
+            <box size="${base_length} ${base_width} ${base_height}"/>
+        </geometry>
+        <origin xyz="0 0 0" rpy="0 0 0"/>
+    </collision>
+    <xacro:box_inertia m="2.5" x="${base_length}" y="${base_width}" z="${base_height}" o_xyz="0 0 0" o_rpy="0 0 0"/>
 </link>
 <xacro:macro name="wheel_link" params="prefix">
@@ -28,4 +35,11 @@
             <material name="grey"/>
         </visual>
+        <collision>
+            <geometry>
+                <sphere radius="${wheel_radius}"/>
+            </geometry>
+            <origin xyz="0 0 0" rpy="0 ${pi/2} ${-pi/2}"/>
+        </collision>
+        <xacro:cylinder_inertia m="0.5" r="${wheel_radius}" h="${wheel_width}" o_xyz="0 0 0" o_rpy="0 0 0"/>
     </link>
 </xacro:macro>
@@ -40,4 +54,11 @@
         <material name="grey"/>
     </visual>
+    <collision>
+        <geometry>
+            <sphere radius="${caster_radius}"/>
+        </geometry>
+        <origin xyz="0 0 0" rpy="0 0 0"/>
+    </collision>
+    <xacro:sphere_inertia m="0.25" r="${caster_radius}" o_xyz="0 0 0" o_rpy="0 0 0"/>
 </link>
 <!-- Joints -->
