Commit message: fixed the code

File: robot_description/urdf/camera.xacro (robot description, xacro)
@@ -25,7 +25,7 @@
 <!-- Joints -->
 <joint name="base_camera_joint" type="fixed">
-    <parent link="base_link"/>
+    <parent link="mobile_base_link"/>
     <child link="camera_link"/>
-    <origin xyz="${(base_length + camera_length) / 2.0} 0 ${base_height / 2.0}" rpy="0 0 0"/>
+    <origin xyz="${(base_length + camera_length) / 2.0} 0 0" rpy="0 0 0"/>
 </joint>
 </robot>

Commit message: updated the code fix for opencv

File: robot_description/urdf/camera.xacro (robot description, xacro)
@@ -1,15 +1,12 @@
 <?xml version="1.0"?>
 <robot xmlns:xacro="http://www.ros.org/wiki/xacro">
-<!-- Include common properties -->
-<xacro:property name="camera_length" value="0.01" />
-<xacro:property name="camera_width" value="0.1" />
-<xacro:property name="camera_height" value="0.05" />
-<!-- Links -->
-   <link name="camera_link">
+    <xacro:property name="camera_length" value="0.01" />
+    <xacro:property name="camera_width" value="0.1" />
+    <xacro:property name="camera_height" value="0.05" />
+    <link name="camera_link">
         <visual>
             <geometry>
                 <box size="${camera_length} ${camera_width} ${camera_height}" />
             </geometry>
-            <origin xyz="0 0 0" rpy="0 0 0" />
             <material name="grey" />
         </visual>
@@ -18,15 +15,19 @@
                 <box size="${camera_length} ${camera_width} ${camera_height}" />
             </geometry>
-            <origin xyz="0 0 0" rpy="0 0 0" />
         </collision>
         <xacro:box_inertia m="0.1" x="${camera_length}" y="${camera_width}" z="${camera_height}"
                            o_xyz="0 0 0" o_rpy="0 0 0" />
     </link>
-<!-- Joints -->
-<joint name="base_camera_joint" type="fixed">
-    <parent link="mobile_base_link"/>
-    <child link="camera_link"/>
-    <origin xyz="${(base_length + camera_length) / 2.0} 0 0" rpy="0 0 0"/>
-</joint>
+    <joint name="base_camera_joint" type="fixed">
+        <parent link="mobile_base_link" />
+        <child link="camera_link" />
+        <origin xyz="${(base_length + camera_length) / 2.0} 0 ${base_height / 2.0}" rpy="0 0 0" />
+    </joint>
+    <link name="camera_link_optical" />
+    <joint name="camera_optical_joint" type="fixed">
+        <origin xyz="0 0 0" rpy="${-pi/2} 0 ${-pi/2}"/>
+        <parent link="camera_link"/>
+        <child link="camera_link_optical"/>
+    </joint>
     <gazebo reference="camera_link">
         <sensor name="camera" type="camera">
