Commit message: modified mobile for collisions

File: robot_description/urdf/mobile_uvc.urdf.xacro (robot description, xacro)
@@ -1,75 +1,133 @@
 <?xml version="1.0"?>
 <robot name="mobile_uvc" xmlns:xacro="http://www.ros.org/wiki/xacro">
-<material name="blue"><color rgba="0 0 1 1"/></material>
-<material name="green"><color rgba="0 1 0 1"/></material>
-<material name="yellow"><color rgba="1 1 0 1"/></material>
-<material name="orange"><color rgba="1 0.5 0 1"/></material>
-<material name="purple"><color rgba="0.5 0 0.5 1"/></material>
-<material name="red"><color rgba="1 0 0 1"/></material>
-<!-- ROOT FRAME -->
-<link name="base_footprint"/>
-<!-- MOBILE ROBOT BODY -->
-<link name="mobile_base_link">
-  <visual>
-    <geometry>
-      <mesh filename="file:///home/linos/cad_projects/mobile/body.stl" scale="0.001 0.001 0.001"/>
-    </geometry>
-    <origin xyz="0.102772 -0.213746 -0.353914" rpy="0 0 0"/>
-    <material name="blue"/>
-  </visual>
-</link>
-<!-- LEFT WHEEL -->
-<link name="left_wheel_link">
-  <visual>
-    <geometry>
-      <mesh filename="file:///home/linos/cad_projects/mobile/left_wheel.stl" scale="0.001 0.001 0.001"/>
-    </geometry>
-    <origin xyz="${0.342038} 0 ${ - 0.119289}" rpy="0 0 0"/>
-    <material name="green"/>
-  </visual>
-</link>
-<!-- RIGHT WHEEL -->
-<link name="right_wheel_link">
-  <visual>
-    <geometry>
-      <mesh filename="file:///home/linos/cad_projects/mobile/right_wheel.stl" scale="0.001 0.001 0.001"/>
-    </geometry>
-    <origin xyz="${- 0.136493} 0 ${ - 0.119289}" rpy="0 0 0"/>
-    <material name="green"/>
-  </visual>
-</link>
-<!-- RODA (third wheel or caster) -->
-<link name="roda_link">
-  <visual>
-    <geometry>
-      <mesh filename="file:///home/linos/cad_projects/mobile/roda.stl" scale="0.001 0.001 0.001"/>
-    </geometry>
-    <origin xyz="0.102772 -0.422475 -0.045338" rpy="0 0 0"/>
-    <material name="green"/>
-  </visual>
-</link>
-<!-- FIXED JOINT BETWEEN FOOTPRINT AND MOBILE BASE -->
-<joint name="base_to_base_footprint_joint" type="fixed">
-  <parent link="base_footprint"/>
-  <child link="mobile_base_link"/>
-  <origin xyz="-0.102772 0.213746 0.353914" rpy="0 0 0"/>
-</joint>
-<joint name="left_wheel_joint" type="continuous">
-  <parent link="mobile_base_link"/>
-  <child link="left_wheel_link"/>
-  <origin xyz="${0.102772 - 0.342038} -0.213746 ${-0.353914 + 0.119289}" rpy="0 0 0"/>
-  <axis xyz="1 0 0"/>
-</joint>
-<joint name="right_wheel_joint" type="continuous">
-  <parent link="mobile_base_link"/>
-  <child link="right_wheel_link"/>
-  <origin xyz="${0.102772 + 0.136493} -0.213746 ${-0.353914 + 0.119289}" rpy="0 0 0"/>
-  <axis xyz="1 0 0"/>
-</joint>
-<joint name="roda_joint" type="continuous">
-  <parent link="mobile_base_link"/>
-  <child link="roda_link"/>
-  <origin xyz="${0.102772 -0.102772} ${-0.213746 +0.422475} ${-0.353914 + 0.045338}" rpy="0 0 0"/>
-  <axis xyz="0 1 0"/>
-</joint>
+  <!-- ========================= -->
+  <!--       PROPERTIES          -->
+  <!-- ========================= -->
+  <!-- Wheel collision radius (all wheels use same radius) -->
+  <xacro:property name="wheel_radius" value="0.119289"/>
+  <xacro:property name="wheel_width" value="0.160767"/>
+  <!-- Roda collision radius -->
+  <xacro:property name="roda_radius" value="0.038463"/>
+  <!-- Base link visual origin -->
+  <xacro:property name="base_x" value="0.102772"/>
+  <xacro:property name="base_y" value="-0.213746"/>
+  <xacro:property name="base_z" value="-0.353914"/>
+  <!-- Wheel visual offsets -->
+  <xacro:property name="left_wheel_x" value="0.342038"/>
+  <xacro:property name="right_wheel_x" value="-0.136493"/>
+  <xacro:property name="wheel_z" value="-0.119289"/>
+  <!-- Roda offsets -->
+  <xacro:property name="roda_x" value="0.102772"/>
+  <xacro:property name="roda_y" value="-0.422475"/>
+  <xacro:property name="roda_z" value="-0.045338"/>
+  <!-- ========================= -->
+  <!--        MATERIALS          -->
+  <!-- ========================= -->
+  <material name="blue"><color rgba="0 0 1 1"/></material>
+  <material name="green"><color rgba="0 1 0 1"/></material>
+  <material name="yellow"><color rgba="1 1 0 1"/></material>
+  <material name="orange"><color rgba="1 0.5 0 1"/></material>
+  <material name="purple"><color rgba="0.5 0 0.5 1"/></material>
+  <material name="red"><color rgba="1 0 0 1"/></material>
+  <!-- ========================= -->
+  <!--        ROOT FRAME         -->
+  <!-- ========================= -->
+  <link name="base_footprint"/>
+  <!-- ========================= -->
+  <!--     MOBILE BASE LINK      -->
+  <!-- ========================= -->
+  <link name="mobile_base_link">
+    <visual>
+      <geometry>
+        <mesh filename="file:///home/linos/cad_projects/mobile/body.stl" scale="0.001 0.001 0.001"/>
+      </geometry>
+      <origin xyz="${base_x} ${base_y} ${base_z}" rpy="0 0 0"/>
+      <material name="blue"/>
+    </visual>
+    <collision>
+      <geometry>
+        <box size=" 0.500 0.849993   0.4 "/>
+      </geometry>
+        <origin xyz="0 0 ${-0.253914/2}" rpy="0 0 0"/>
+    </collision>
+  </link>
+  <!-- ========================= -->
+  <!--       LEFT WHEEL          -->
+  <!-- ========================= -->
+  <link name="left_wheel_link">
+    <visual>
+      <geometry>
+        <mesh filename="file:///home/linos/cad_projects/mobile/left_wheel.stl" scale="0.001 0.001 0.001"/>
+      </geometry>
+      <origin xyz="${left_wheel_x} 0 ${wheel_z}" rpy="0 0 0"/>
+      <material name="green"/>
+    </visual>
+    <collision>
+      <geometry>
+        <sphere radius="${wheel_radius}"/>
+      </geometry>
+      <origin xyz="${wheel_width/2} 0 0" rpy="0 0 0"/>
+    </collision>
+  </link>
+  <!-- ========================= -->
+  <!--       RIGHT WHEEL         -->
+  <!-- ========================= -->
+  <link name="right_wheel_link">
+    <visual>
+      <geometry>
+        <mesh filename="file:///home/linos/cad_projects/mobile/right_wheel.stl" scale="0.001 0.001 0.001"/>
+      </geometry>
+      <origin xyz="${right_wheel_x} 0 ${wheel_z}" rpy="0 0 0"/>
+      <material name="green"/>
+    </visual>
+    <collision>
+      <geometry>
+        <sphere radius="${wheel_radius}"/>
+      </geometry>
+      <origin xyz="${-wheel_width/2} 0 0" rpy="0 0 0"/>
+    </collision>
+  </link>
+  <!-- ========================= -->
+  <!--           RODA            -->
+  <!-- ========================= -->
+  <link name="roda_link">
+    <visual>
+      <geometry>
+        <mesh filename="file:///home/linos/cad_projects/mobile/roda.stl" scale="0.001 0.001 0.001"/>
+      </geometry>
+      <origin xyz="${roda_x} ${roda_y} ${roda_z}" rpy="0 0 0"/>
+      <material name="green"/>
+    </visual>
+    <collision>
+      <geometry>
+        <sphere radius="${roda_radius}"/>
+      </geometry>
+    </collision>
+  </link>
+  <!-- ========================= -->
+  <!--           JOINTS          -->
+  <!-- ========================= -->
+  <joint name="base_to_base_footprint_joint" type="fixed">
+    <parent link="base_footprint"/>
+    <child link="mobile_base_link"/>
+    <origin xyz="${-base_x} ${-base_y} ${-base_z}" rpy="0 0 0"/>
+  </joint>
+  <joint name="left_wheel_joint" type="continuous">
+    <parent link="mobile_base_link"/>
+    <child link="left_wheel_link"/>
+    <origin xyz="${base_x - left_wheel_x} ${base_y} ${base_z - wheel_z}" rpy="0 0 0"/>
+    <axis xyz="1 0 0"/>
+  </joint>
+  <joint name="right_wheel_joint" type="continuous">
+    <parent link="mobile_base_link"/>
+    <child link="right_wheel_link"/>
+    <origin xyz="${base_x - right_wheel_x} ${base_y} ${base_z - wheel_z}" rpy="0 0 0"/>
+    <axis xyz="1 0 0"/>
+  </joint>
+  <joint name="roda_joint" type="continuous">
+    <parent link="mobile_base_link"/>
+    <child link="roda_link"/>
+    <origin xyz="${base_x - roda_x} ${base_y - roda_y} ${base_z - roda_z}" rpy="0 0 0"/>
+    <axis xyz="0 1 0"/>
+  </joint>
 </robot>
