Commit message: Initialize common material properties for URDF modules

File: robot_description/urdf/common_properties.xacro (robot description, xacro)
@@ -1,3 +1,16 @@
-<? xml version="1.0"?>
-<robot xmlns:xacro="http://www.ros.org/wiki/xacro">
+<?xml version="1.0"?>
+<robot name="common_properties" xmlns:xacro="http://www.ros.org/wiki/xacro">
+    <!-- Common materials -->
+    <material name="blue">
+        <color rgba="0 0 0.8 1"/>
+    </material>
+    <material name="grey">
+        <color rgba="0.5 0.5 0.5 1"/>
+    </material>
+    <material name="yellow">
+        <color rgba="0.8 0.8 0 1"/>
+    </material>
+    <material name="orange">
+        <color rgba="0.8 0.4 0 1"/>
+    </material>
 </robot>

Commit message: Add inertia properties

File: robot_description/urdf/common_properties.xacro (robot description, xacro)
@@ -14,3 +14,22 @@
         <color rgba="0.8 0.4 0 1"/>
     </material>
+    <!-- Common inertia calculations -->
+    <xacro:property name="box_inertia" params="m x y z o_xyz o_rpy">
+        <inertia
+            ixx="${(1/12.0)*m*(y**2 + z**2)}" ixy="0" ixz="0"
+            iyy="${(1/12.0)*m*(x**2 + z**2)}" iyz="0"
+            izz="${(1/12.0)*m*(x**2 + y**2)}"/>
+    </xacro:property>
+    <xacro:property name="cylinder_inertia" params="m r h o_xyz o_rpy">
+        <inertia
+            ixx="${(1/12.0)*m*(3*r**2 + h**2)}" ixy="0" ixz="0"
+            iyy="${(1/12.0)*m*(3*r**2 + h**2)}" iyz="0"
+            izz="${(1/2.0)*m*r**2}"/>
+    </xacro:property>
+    <xacro:property name="sphere_inertia" params="m r o_xyz o_rpy">
+        <inertia
+            ixx="${(2/5.0)*m*r**2}" ixy="0" ixz="0"
+            iyy="${(2/5.0)*m*r**2}" iyz="0"
+            izz="${(2/5.0)*m*r**2}"/>
+    </xacro:property>
 </robot>

Commit message: fixed inetia features

File: robot_description/urdf/common_properties.xacro (robot description, xacro)
@@ -15,21 +15,27 @@
     </material>
     <!-- Common inertia calculations -->
-    <xacro:property name="box_inertia" params="m x y z o_xyz o_rpy">
+    <xacro:macro name="box_inertia" params="m x y z o_xyz o_rpy">
+        <mass value="${m}"/>
+        <origin xyz="${o_xyz}" rpy="${o_rpy}"/>
         <inertia
-            ixx="${(1/12.0)*m*(y**2 + z**2)}" ixy="0" ixz="0"
-            iyy="${(1/12.0)*m*(x**2 + z**2)}" iyz="0"
-            izz="${(1/12.0)*m*(x**2 + y**2)}"/>
-    </xacro:property>
-    <xacro:property name="cylinder_inertia" params="m r h o_xyz o_rpy">
+            ixx="${(1/12.0)*m*(y*y + z*z)}" ixy="0" ixz="0"
+            iyy="${(1/12.0)*m*(x*x + z*z)}" iyz="0"
+            izz="${(1/12.0)*m*(x*x + y*y)}"/>
+    </xacro:macro>
+    <xacro:macro name="cylinder_inertia" params="m r h o_xyz o_rpy">
+        <mass value="${m}"/>
+        <origin xyz="${o_xyz}" rpy="${o_rpy}"/>
         <inertia
-            ixx="${(1/12.0)*m*(3*r**2 + h**2)}" ixy="0" ixz="0"
-            iyy="${(1/12.0)*m*(3*r**2 + h**2)}" iyz="0"
-            izz="${(1/2.0)*m*r**2}"/>
-    </xacro:property>
-    <xacro:property name="sphere_inertia" params="m r o_xyz o_rpy">
+            ixx="${(1/12.0)*m*(3*r*r + h*h)}" ixy="0" ixz="0"
+            iyy="${(1/12.0)*m*(3*r*r + h*h)}" iyz="0"
+            izz="${(1/2.0)*m*r*r}"/>
+    </xacro:macro>
+    <xacro:macro name="sphere_inertia" params="m r o_xyz o_rpy">
+        <mass value="${m}"/>
+        <origin xyz="${o_xyz}" rpy="${o_rpy}"/>
         <inertia
-            ixx="${(2/5.0)*m*r**2}" ixy="0" ixz="0"
-            iyy="${(2/5.0)*m*r**2}" iyz="0"
-            izz="${(2/5.0)*m*r**2}"/>
-    </xacro:property>
+            ixx="${(2/5.0)*m*r*r}" ixy="0" ixz="0"
+            iyy="${(2/5.0)*m*r*r}" iyz="0"
+            izz="${(2/5.0)*m*r*r}"/>
+    </xacro:macro>
 </robot>

Commit message: fixed inertia issues

File: robot_description/urdf/common_properties.xacro (robot description, xacro)
@@ -16,26 +16,31 @@
     <!-- Common inertia calculations -->
     <xacro:macro name="box_inertia" params="m x y z o_xyz o_rpy">
-        <mass value="${m}"/>
-        <origin xyz="${o_xyz}" rpy="${o_rpy}"/>
-        <inertia
-            ixx="${(1/12.0)*m*(y*y + z*z)}" ixy="0" ixz="0"
-            iyy="${(1/12.0)*m*(x*x + z*z)}" iyz="0"
-            izz="${(1/12.0)*m*(x*x + y*y)}"/>
+        <inertial>
+            <mass value="${m}" />
+            <origin xyz="${o_xyz}" rpy="${o_rpy}" />
+            <inertia ixx="${(m/12) * (y*y + z*z)}" ixy="0" ixz="0"
+                     iyy="${(m/12) * (x*x + z*z)}" iyz="0"
+                     izz="${(m/12) * (x*x + y*y)}" />
+        </inertial>
     </xacro:macro>
     <xacro:macro name="cylinder_inertia" params="m r h o_xyz o_rpy">
-        <mass value="${m}"/>
-        <origin xyz="${o_xyz}" rpy="${o_rpy}"/>
-        <inertia
-            ixx="${(1/12.0)*m*(3*r*r + h*h)}" ixy="0" ixz="0"
-            iyy="${(1/12.0)*m*(3*r*r + h*h)}" iyz="0"
-            izz="${(1/2.0)*m*r*r}"/>
+        <inertial>
+            <mass value="${m}"/>
+            <origin xyz="${o_xyz}" rpy="${o_rpy}"/>
+            <inertia
+                ixx="${(1/12.0)*m*(3*r*r + h*h)}" ixy="0" ixz="0"
+                iyy="${(1/12.0)*m*(3*r*r + h*h)}" iyz="0"
+                izz="${(1/2.0)*m*r*r}"/>
+        </inertial>
     </xacro:macro>
     <xacro:macro name="sphere_inertia" params="m r o_xyz o_rpy">
-        <mass value="${m}"/>
-        <origin xyz="${o_xyz}" rpy="${o_rpy}"/>
-        <inertia
-            ixx="${(2/5.0)*m*r*r}" ixy="0" ixz="0"
-            iyy="${(2/5.0)*m*r*r}" iyz="0"
-            izz="${(2/5.0)*m*r*r}"/>
+        <inertial>
+            <mass value="${m}"/>
+            <origin xyz="${o_xyz}" rpy="${o_rpy}"/>
+            <inertia
+                ixx="${(2/5.0)*m*r*r}" ixy="0" ixz="0"
+                iyy="${(2/5.0)*m*r*r}" iyz="0"
+                izz="${(2/5.0)*m*r*r}"/>
+        </inertial>
     </xacro:macro>
 </robot>

Commit message: fixed the code

File: robot_description/urdf/common_properties.xacro (robot description, xacro)
@@ -2,16 +2,11 @@
 <robot xmlns:xacro="http://www.ros.org/wiki/xacro">
     <!-- Common materials -->
-    <material name="blue">
-        <color rgba="0 0 0.8 1"/>
-    </material>
-    <material name="grey">
-        <color rgba="0.5 0.5 0.5 1"/>
-    </material>
-    <material name="yellow">
-        <color rgba="0.8 0.8 0 1"/>
-    </material>
-    <material name="orange">
-        <color rgba="0.8 0.4 0 1"/>
-    </material>
+    <material name="blue"><color rgba="0 0 1 1"/></material>
+    <material name="green"><color rgba="0 1 0 1"/></material>
+    <material name="yellow"><color rgba="1 1 0 1"/></material>
+    <material name="orange"><color rgba="1 0.5 0 1"/></material>
+    <material name="purple"><color rgba="0.5 0 0.5 1"/></material>
+    <material name="red"><color rgba="1 0 0 1"/></material>
+    <material name="gray"><color rgba="0.5 0.5 0.5 1"/></material>
     <!-- Common inertia calculations -->
     <xacro:macro name="box_inertia" params="m x y z o_xyz o_rpy">
