Commit message: modified the code

File: robot_description/urdf/scara_arm.xacro (robot description, xacro)
@@ -1,12 +1,7 @@
 <?xml version="1.0"?>
-<robot name="gripper_scara" xmlns:xacro="http://www.ros.org/wiki/xacro">
-<material name="blue"><color rgba="0 0 1 1"/></material>
-<material name="green"><color rgba="0 1 0 1"/></material>
-<material name="yellow"><color rgba="1 1 0 1"/></material>
-<material name="orange"><color rgba="1 0.5 0 1"/></material>
-<material name="purple"><color rgba="0.5 0 0.5 1"/></material>
-<material name="red"><color rgba="1 0 0 1"/></material>
-<link name="base_footprint"/>
+<robot xmlns:xacro="http://www.ros.org/wiki/xacro">
+<!-- ========================= -->
 <!-- BASE LINK -->
+<!-- ========================= -->
 <link name="gripper_base_link">
   <visual>
@@ -17,10 +12,12 @@
     <material name="blue"/>
   </visual>
+  <!-- CYLINDER COLLISION -->
   <collision>
     <origin xyz="0.04 ${0.0402/2-0.02} ${0.02}" rpy="${pi} 0 0"/>
     <geometry>
-      <cylinder radius="${0.06}" length="0.06"/>
-    </geometry>
-  </collision>
+      <cylinder radius="0.06" length="0.06"/>
+    </geometry>
+  </collision>
+  <!-- BOX COLLISION -->
   <collision>
     <origin xyz="0.008 0 0.21" rpy="${pi} 0 0"/>
@@ -29,16 +26,22 @@
     </geometry>
   </collision>
-  <inertial>
-    <!-- match the main collision frame rotation -->
-    <origin xyz="0.0164 0.0 0.16" rpy="${pi} 0 0"/>
-    <mass value="3.0"/>
-    <inertia
-      ixx="0.0353"
-      iyy="0.0348"
-      izz="0.00377"
-      ixy="0.0" ixz="0.0" iyz="0.0"/>
-  </inertial>
-</link>
+  <!-- INERTIA USING MACROS -->
+  <xacro:cylinder_inertia
+      m="0.8"
+      r="0.06"
+      h="0.06"
+      o_xyz="0.04 ${0.0402/2-0.02} 0.02"
+      o_rpy="${pi} 0 0"/>
+  <xacro:box_inertia
+      m="2.2"
+      x="0.06"
+      y="0.1"
+      z="0.317"
+      o_xyz="0.008 0 0.21"
+      o_rpy="${pi} 0 0"/>
+</link>
+<!-- ========================= -->
 <!-- SLIDER -->
+<!-- ========================= -->
 <link name="slider_carriage_link">
   <visual>
@@ -46,5 +49,5 @@
       <mesh filename="file:///home/linos/cad_projects/gripper/slider_carriage.stl" scale="0.001 0.001 0.001"/>
     </geometry>
-    <origin xyz="0 ${-0.0342/2} ${0.253}" rpy="0 0 0"/>
+    <origin xyz="0 ${-0.0342/2} 0.253" rpy="0 0 0"/>
     <material name="green"/>
   </visual>
@@ -55,15 +58,15 @@
     <origin xyz="0.07 0 0.01" rpy="0 0 0"/>
   </collision>
-  <inertial>
-    <origin xyz="0.07 0 0.01" rpy="0 0 0"/>
-    <mass value="0.6"/>
-    <inertia
-      ixx="0.000325"
-      iyy="0.000425"
-      izz="0.00026"
-      ixy="0.0" ixz="0.0" iyz="0.0"/>
-  </inertial>
-</link>
+  <xacro:box_inertia
+      m="0.6"
+      x="0.06"
+      y="0.04"
+      z="0.07"
+      o_xyz="0.07 0 0.01"
+      o_rpy="0 0 0"/>
+</link>
+<!-- ========================= -->
 <!-- SHOULDER -->
+<!-- ========================= -->
 <link name="shoulder_link">
   <visual>
@@ -80,15 +83,15 @@
     <origin xyz="0.06 0.03 0.01" rpy="0 0 ${pi/7}"/>
   </collision>
-  <inertial>
-    <origin xyz="0.06 0.03 0.01" rpy="0 0 ${pi/7}"/>
-    <mass value="0.5"/>
-    <inertia
-      ixx="0.000205"
-      iyy="0.000812"
-      izz="0.000653"
-      ixy="0.0" ixz="0.0" iyz="0.0"/>
-  </inertial>
-</link>
+  <xacro:box_inertia
+      m="0.5"
+      x="0.123"
+      y="0.0235"
+      z="0.066"
+      o_xyz="0.06 0.03 0.01"
+      o_rpy="0 0 ${pi/7}"/>
+</link>
+<!-- ========================= -->
 <!-- ELBOW -->
+<!-- ========================= -->
 <link name="elbow_link">
   <visual>
@@ -105,15 +108,15 @@
     <origin xyz="0.016 -0.05 0.01" rpy="0 0 -1.25"/>
   </collision>
-  <inertial>
-    <origin xyz="0.016 -0.05 0.01" rpy="0 0 -1.25"/>
-    <mass value="0.4"/>
-    <inertia
-      ixx="0.000170"
-      iyy="0.000650"
-      izz="0.000529"
-      ixy="0.0" ixz="0.0" iyz="0.0"/>
-  </inertial>
-</link>
+  <xacro:box_inertia
+      m="0.4"
+      x="0.123"
+      y="0.027"
+      z="0.066"
+      o_xyz="0.016 -0.05 0.01"
+      o_rpy="0 0 -1.25"/>
+</link>
+<!-- ========================= -->
 <!-- WRIST -->
+<!-- ========================= -->
 <link name="wrist_link">
   <visual>
@@ -130,15 +133,15 @@
     <origin xyz="0 0 -0.02" rpy="${-pi/2} 0 0"/>
   </collision>
-  <inertial>
-    <origin xyz="0 0 -0.02" rpy="${-pi/2} 0 0"/>
-    <mass value="0.4"/>
-    <inertia
-      ixx="0.000108"
-      iyy="0.000096"
-      izz="0.000138"
-      ixy="0.0" ixz="0.0" iyz="0.0"/>
-  </inertial>
-</link>
+  <xacro:box_inertia
+      m="0.4"
+      x="0.055"
+      y="0.06"
+      z="0.04"
+      o_xyz="0 0 -0.02"
+      o_rpy="${-pi/2} 0 0"/>
+</link>
+<!-- ========================= -->
 <!-- LEFT FINGER -->
+<!-- ========================= -->
 <link name="left_finger_link">
   <visual>
@@ -155,15 +158,15 @@
     <origin xyz="0 0.02 -0.02" rpy="0 ${pi} 0"/>
   </collision>
-  <inertial>
-    <origin xyz="0 0.02 -0.02" rpy="0 ${pi} 0"/>
-    <mass value="0.08"/>
-    <inertia
-      ixx="0.0000198"
-      iyy="0.0000126"
-      izz="0.0000111"
-      ixy="0.0" ixz="0.0" iyz="0.0"/>
-  </inertial>
-</link>
+  <xacro:box_inertia
+      m="0.08"
+      x="0.017"
+      y="0.037"
+      z="0.04"
+      o_xyz="0 0.02 -0.02"
+      o_rpy="0 ${pi} 0"/>
+</link>
+<!-- ========================= -->
 <!-- RIGHT FINGER -->
+<!-- ========================= -->
 <link name="right_finger_link">
   <visual>
@@ -180,17 +183,15 @@
     <origin xyz="0 0.02 -0.02" rpy="0 ${pi} 0"/>
   </collision>
-  <inertial>
-    <origin xyz="0 0.02 -0.02" rpy="0 ${pi} 0"/>
-    <mass value="0.08"/>
-    <inertia
-      ixx="0.0000198"
-      iyy="0.0000126"
-      izz="0.0000111"
-      ixy="0.0" ixz="0.0" iyz="0.0"/>
-  </inertial>
+  <xacro:box_inertia
+      m="0.08"
+      x="0.017"
+      y="0.037"
+      z="0.04"
+      o_xyz="0 0.02 -0.02"
+      o_rpy="0 ${pi} 0"/>
 </link>
 <!-- JOINTS (unchanged) -->
-<joint name="base_to_footprint" type="fixed">
-  <parent link="base_footprint"/>
+<joint name="arm_base_to_mobile_base" type="fixed">
+  <parent link="mobile_uvc_base_link"/>
   <child link="gripper_base_link"/>
   <origin xyz="0 0 0" rpy="0 0 0"/>
@@ -215,5 +216,5 @@
   <origin xyz="0.095 0.047 0" rpy="0 0 0"/>
   <axis xyz="0 0 1"/>
-  <limit lower="${0}" upper="${3.343}" effort="50" velocity="1.0"/>
+  <limit lower="0" upper="3.343" effort="50" velocity="1.0"/>
 </joint>
 <joint name="wrist_to_elbow" type="revolute">

Commit message: add new model

File: robot_description/urdf/scara_arm.xacro (robot description, xacro)
@@ -1,241 +1,67 @@
 <?xml version="1.0"?>
 <robot xmlns:xacro="http://www.ros.org/wiki/xacro">
-<!-- ========================= -->
-<!-- BASE LINK -->
-<!-- ========================= -->
-<link name="gripper_base_link">
+<xacro:property name="base_cylinder_height" value="0.060"/>
+<xacro:property name="base_cylinder_radius" value="0.12"/>
+<xacro:property name="mass_base_cylinder" value="1.5"/>
+<xacro:property name="mass_rotary_bearing" value="1.0"/>
+<xacro:property name="mass_waist_structure" value="3.0"/>
+<xacro:property name="mass_slider_carriage" value="1.8"/>
+<xacro:property name="mass_shoulder" value="2.0"/>
+<xacro:property name="mass_elbow" value="1.7"/>
+<xacro:property name="mass_wrist" value="1.1"/>
+<xacro:property name="mass_finger" value="0.25"/>
+<link name="arm_base_link">
   <visual>
     <geometry>
-      <mesh filename="file:///home/linos/cad_projects/gripper/base.stl" scale="0.001 0.001 0.001"/>
+      <mesh filename="file:///home/linos/cad_projects/gripper/v1.2/base.stl" scale="0.001 0.001 0.001"/>
     </geometry>
-    <origin xyz="0 ${0.0402/2} ${0.04-0.01}" rpy="${pi} 0 0"/>
-    <material name="blue"/>
-  </visual>
-  <!-- CYLINDER COLLISION -->
-  <collision>
-    <origin xyz="0.04 ${0.0402/2-0.02} ${0.02}" rpy="${pi} 0 0"/>
-    <geometry>
-      <cylinder radius="0.06" length="0.06"/>
-    </geometry>
-  </collision>
-  <!-- BOX COLLISION -->
-  <collision>
-    <origin xyz="0.008 0 0.21" rpy="${pi} 0 0"/>
-    <geometry>
-      <box size="0.06 0.1 0.317"/>
-    </geometry>
-  </collision>
-  <!-- INERTIA USING MACROS -->
-  <xacro:cylinder_inertia
-      m="0.8"
-      r="0.06"
-      h="0.06"
-      o_xyz="0.04 ${0.0402/2-0.02} 0.02"
-      o_rpy="${pi} 0 0"/>
-  <xacro:box_inertia
-      m="2.2"
-      x="0.06"
-      y="0.1"
-      z="0.317"
-      o_xyz="0.008 0 0.21"
-      o_rpy="${pi} 0 0"/>
-</link>
-<!-- ========================= -->
-<!-- SLIDER -->
-<!-- ========================= -->
-<link name="slider_carriage_link">
-  <visual>
-    <geometry>
-      <mesh filename="file:///home/linos/cad_projects/gripper/slider_carriage.stl" scale="0.001 0.001 0.001"/>
-    </geometry>
-    <origin xyz="0 ${-0.0342/2} 0.253" rpy="0 0 0"/>
-    <material name="green"/>
+    <origin xyz="0 0 0" rpy="0 0 0"/>
+    <material name="gray"/>
   </visual>
   <collision>
     <geometry>
-      <box size="0.06 0.04 0.07"/>
+      <cylinder radius="${base_cylinder_radius}" length="${base_cylinder_height}"/>
     </geometry>
-    <origin xyz="0.07 0 0.01" rpy="0 0 0"/>
   </collision>
-  <xacro:box_inertia
-      m="0.6"
-      x="0.06"
-      y="0.04"
-      z="0.07"
-      o_xyz="0.07 0 0.01"
+  <xacro:cylinder_inertia
+      m="${mass_base_cylinder}"
+      r="${base_cylinder_radius}"
+      h="${base_cylinder_height}"
+      o_xyz="0 0 0"
       o_rpy="0 0 0"/>
 </link>
-<!-- ========================= -->
-<!-- SHOULDER -->
-<!-- ========================= -->
-<link name="shoulder_link">
+<link name="waist_link">
   <visual>
     <geometry>
-      <mesh filename="file:///home/linos/cad_projects/gripper/shoulder.stl" scale="0.001 0.001 0.001"/>
+      <mesh filename="file:///home/linos/cad_projects/gripper/v1.2/waist.stl" scale="0.001 0.001 0.001"/>
     </geometry>
-    <origin xyz="-0.08 ${-0.0342/2} 0.253" rpy="0 0 0"/>
+    <origin xyz="0 0 ${-base_cylinder_height}" rpy="0 0 0"/>
     <material name="yellow"/>
   </visual>
   <collision>
     <geometry>
-      <box size="0.123 0.0235 0.066"/>
+      <box size="0.06 0.10 0.317"/>
     </geometry>
-    <origin xyz="0.06 0.03 0.01" rpy="0 0 ${pi/7}"/>
+    <origin xyz="0 0 0" rpy="0 0 0"/>
   </collision>
   <xacro:box_inertia
-      m="0.5"
-      x="0.123"
-      y="0.0235"
-      z="0.066"
-      o_xyz="0.06 0.03 0.01"
-      o_rpy="0 0 ${pi/7}"/>
+      m="${mass_rotary_bearing + mass_waist_structure}"
+      x="0.06"
+      y="0.10"
+      z="0.317"
+      o_xyz="0 0 0"
+      o_rpy="0 0 0"/>
 </link>
-<!-- ========================= -->
-<!-- ELBOW -->
-<!-- ========================= -->
-<link name="elbow_link">
-  <visual>
-    <geometry>
-      <mesh filename="file:///home/linos/cad_projects/gripper/elbow.stl" scale="0.001 0.001 0.001"/>
-    </geometry>
-    <origin xyz="-0.18 -0.047 0.253" rpy="0 0 0"/>
-    <material name="orange"/>
-  </visual>
-  <collision>
-    <geometry>
-      <box size="0.123 0.027 0.066"/>
-    </geometry>
-    <origin xyz="0.016 -0.05 0.01" rpy="0 0 -1.25"/>
-  </collision>
-  <xacro:box_inertia
-      m="0.4"
-      x="0.123"
-      y="0.027"
-      z="0.066"
-      o_xyz="0.016 -0.05 0.01"
-      o_rpy="0 0 -1.25"/>
-</link>
-<!-- ========================= -->
-<!-- WRIST -->
-<!-- ========================= -->
-<link name="wrist_link">
-  <visual>
-    <geometry>
-      <mesh filename="file:///home/linos/cad_projects/gripper/wrist.stl" scale="0.001 0.001 0.001"/>
-    </geometry>
-    <origin xyz="-0.0275 -0.02 -0.03" rpy="${-pi/2} 0 0"/>
-    <material name="purple"/>
-  </visual>
-  <collision>
-    <geometry>
-      <box size="0.055 0.06 0.04"/>
-    </geometry>
-    <origin xyz="0 0 -0.02" rpy="${-pi/2} 0 0"/>
-  </collision>
-  <xacro:box_inertia
-      m="0.4"
-      x="0.055"
-      y="0.06"
-      z="0.04"
-      o_xyz="0 0 -0.02"
-      o_rpy="${-pi/2} 0 0"/>
-</link>
-<!-- ========================= -->
-<!-- LEFT FINGER -->
-<!-- ========================= -->
-<link name="left_finger_link">
-  <visual>
-    <geometry>
-      <mesh filename="file:///home/linos/cad_projects/gripper/left_finger.stl" scale="0.001 0.001 0.001"/>
-    </geometry>
-    <origin xyz="0.16 0.117 -0.155" rpy="0 ${pi} ${pi/12}"/>
-    <material name="red"/>
-  </visual>
-  <collision>
-    <geometry>
-      <box size="0.017 0.037 0.04"/>
-    </geometry>
-    <origin xyz="0 0.02 -0.02" rpy="0 ${pi} 0"/>
-  </collision>
-  <xacro:box_inertia
-      m="0.08"
-      x="0.017"
-      y="0.037"
-      z="0.04"
-      o_xyz="0 0.02 -0.02"
-      o_rpy="0 ${pi} 0"/>
-</link>
-<!-- ========================= -->
-<!-- RIGHT FINGER -->
-<!-- ========================= -->
-<link name="right_finger_link">
-  <visual>
-    <geometry>
-      <mesh filename="file:///home/linos/cad_projects/gripper/right_finger.stl" scale="0.001 0.001 0.001"/>
-    </geometry>
-    <origin xyz="0.215 0.117 -0.155" rpy="0 ${pi} ${pi/12}"/>
-    <material name="red"/>
-  </visual>
-  <collision>
-    <geometry>
-      <box size="0.017 0.037 0.04"/>
-    </geometry>
-    <origin xyz="0 0.02 -0.02" rpy="0 ${pi} 0"/>
-  </collision>
-  <xacro:box_inertia
-      m="0.08"
-      x="0.017"
-      y="0.037"
-      z="0.04"
-      o_xyz="0 0.02 -0.02"
-      o_rpy="0 ${pi} 0"/>
-</link>
-<!-- JOINTS (unchanged) -->
-<joint name="arm_base_to_mobile_base" type="fixed">
+<joint name="arm_base_to_mobile_base_link" type="fixed">
   <parent link="mobile_uvc_base_link"/>
-  <child link="gripper_base_link"/>
+  <child link="arm_base_link"/>
   <origin xyz="0 0 0" rpy="0 0 0"/>
 </joint>
-<joint name="slider_to_base" type="prismatic">
-  <parent link="gripper_base_link"/>
-  <child link="slider_carriage_link"/>
-  <origin xyz="0 0 ${0.253}" rpy="0 0 0"/>
+<joint name="arm_base_to_waist" type="revolute">
+  <parent link="arm_base_link"/>
+  <child link="waist_link"/>
+  <origin xyz="0 0 ${base_cylinder_height}" rpy="0 0 0"/>
   <axis xyz="0 0 1"/>
-  <limit lower="0" upper="-0.15" effort="50" velocity="0.1"/>
-</joint>
-<joint name="shoulder_to_slider" type="revolute">
-  <parent link="slider_carriage_link"/>
-  <child link="shoulder_link"/>
-  <origin xyz="0.08 0 ${0.263/2 -0.1315}" rpy="0 0 0"/>
-  <axis xyz="0 0 1"/>
-  <limit lower="${-pi/2}" upper="${pi/4}" effort="50" velocity="1.0"/>
-</joint>
-<joint name="elbow_to_shoulder" type="revolute">
-  <parent link="shoulder_link"/>
-  <child link="elbow_link"/>
-  <origin xyz="0.095 0.047 0" rpy="0 0 0"/>
-  <axis xyz="0 0 1"/>
-  <limit lower="0" upper="3.343" effort="50" velocity="1.0"/>
-</joint>
-<joint name="wrist_to_elbow" type="revolute">
-  <parent link="elbow_link"/>
-  <child link="wrist_link"/>
-  <origin xyz="0.025 -0.088 0" rpy="0 0 0"/>
-  <axis xyz="0 0 1"/>
-  <limit lower="${-pi/2}" upper="${pi/2}" effort="50" velocity="1.0"/>
-</joint>
-<joint name="left_finger_to_wrist" type="prismatic">
-  <parent link="wrist_link"/>
-  <child link="left_finger_link"/>
-  <origin xyz="0.0275 -0.02 -0.05" rpy="0 0 0"/>
-  <axis xyz="1 0 0"/>
-  <limit lower="-0.015" upper="0.015" effort="20" velocity="0.05"/>
-</joint>
-<joint name="right_finger_to_wrist" type="prismatic">
-  <parent link="wrist_link"/>
-  <child link="right_finger_link"/>
-  <origin xyz="-0.02 -0.02 -0.05" rpy="0 0 0"/>
-  <axis xyz="1 0 0"/>
-  <limit lower="-0.015" upper="0.015" effort="20" velocity="0.05"/>
+  <limit lower="${-pi* 5/6}" upper="${pi*5/6}" effort="50" velocity="1.0"/>
 </joint>
 </robot>

Commit message: add new link and joint

File: robot_description/urdf/scara_arm.xacro (robot description, xacro)
@@ -3,4 +3,5 @@
 <xacro:property name="base_cylinder_height" value="0.060"/>
 <xacro:property name="base_cylinder_radius" value="0.12"/>
+<xacro:property name="slider_length" value="0.472"/>
 <xacro:property name="mass_base_cylinder" value="1.5"/>
 <xacro:property name="mass_rotary_bearing" value="1.0"/>
@@ -53,4 +54,26 @@
       o_rpy="0 0 0"/>
 </link>
+<link name="slide_carriage_link">
+  <visual>
+    <geometry>
+      <mesh filename="file:///home/linos/cad_projects/gripper/v1.2/slider_carriage.stl" scale="0.001 0.001 0.001"/>
+    </geometry>
+    <origin xyz="0 0 ${-slider_length - base_cylinder_height}" rpy="0 0 0"/>
+    <material name="green"/>
+  </visual>
+  <collision>
+    <geometry>
+      <box size="0.06 0.04 0.07"/>
+    </geometry>
+    <origin xyz="0 0 0" rpy="0 0 0"/>
+  </collision>
+  <xacro:box_inertia
+      m="${mass_slider_carriage}"
+      x="0.06"
+      y="0.04"
+      z="0.07"
+      o_xyz="0 0 0"
+      o_rpy="0 0 0"/>
+</link>
 <joint name="arm_base_to_mobile_base_link" type="fixed">
   <parent link="mobile_uvc_base_link"/>
@@ -65,3 +88,10 @@
   <limit lower="${-pi* 5/6}" upper="${pi*5/6}" effort="50" velocity="1.0"/>
 </joint>
+<joint name="slide_carriage_to_slider" type="prismatic">
+  <parent link="waist_link"/>
+  <child link="slide_carriage_link"/>
+  <origin xyz="0 0 ${base_cylinder_height + slider_length - 0.09 + 0.05}" rpy="0 0 0"/>
+  <axis xyz="0 0 1"/>
+  <limit lower="${-slider_length + 0.126}" upper="${0}" effort="50" velocity="0.1"/>
+</joint>
 </robot>

Commit message: add new link

File: robot_description/urdf/scara_arm.xacro (robot description, xacro)
@@ -76,4 +76,26 @@
       o_rpy="0 0 0"/>
 </link>
+<link name="shoulder_link">
+  <visual>
+    <geometry>
+      <mesh filename="file:///home/linos/cad_projects/gripper/v1.2/shoulder.stl" scale="0.001 0.001 0.001"/>
+    </geometry>
+    <origin xyz="0 -0.1212 ${-slider_length + base_cylinder_height - 2 * 0.09}" rpy="0 0 0"/>
+    <material name="orange"/>
+  </visual>
+  <collision>
+    <geometry>
+      <box size="0.12 0.04 0.06"/>
+    </geometry>
+    <origin xyz="0 0 0" rpy="0 0 0"/>
+  </collision>
+  <xacro:box_inertia
+      m="${mass_shoulder}"
+      x="0.12"
+      y="0.04"
+      z="0.06"
+      o_xyz="0 0 0"
+      o_rpy="0 0 0"/>
+</link>
 <joint name="arm_base_to_mobile_base_link" type="fixed">
   <parent link="mobile_uvc_base_link"/>
@@ -95,3 +117,10 @@
   <limit lower="${-slider_length + 0.126}" upper="${0}" effort="50" velocity="0.1"/>
 </joint>
+<joint name="shoulder_to_slide_carriage" type="revolute">
+  <parent link="slide_carriage_link"/>
+  <child link="shoulder_link"/>
+  <origin xyz="0 0.12124 0.06" rpy="0 0 0"/>
+  <axis xyz="0 1 0"/>
+  <limit lower="${-pi/2}" upper="${pi/2}" effort="50" velocity="1.0"/>
+</joint>
 </robot>

Commit message: add new link

File: robot_description/urdf/scara_arm.xacro (robot description, xacro)
@@ -88,8 +88,30 @@
       <box size="0.12 0.04 0.06"/>
     </geometry>
+    <origin xyz="0 -0.358 ${-slider_length + base_cylinder_height - 2 * 0.09}" rpy="0 0 0"/>
+  </collision>
+  <xacro:box_inertia
+      m="${mass_shoulder}"
+      x="0.12"
+      y="0.04"
+      z="0.06"
+      o_xyz="0 0 0"
+      o_rpy="0 0 0"/>
+</link>
+<link name="elbow_link">
+  <visual>
+    <geometry>
+      <mesh filename="file:///home/linos/cad_projects/gripper/v1.2/elbow.stl" scale="0.001 0.001 0.001"/>
+    </geometry>
+    <origin xyz="0 ${-0.48} ${-slider_length + base_cylinder_height - 2 * 0.09}" rpy="0 0 0"/>
+    <material name="red"/>
+  </visual>
+  <collision>
+    <geometry>
+      <box size="0.12 0.04 0.06"/>
+    </geometry>
     <origin xyz="0 0 0" rpy="0 0 0"/>
   </collision>
   <xacro:box_inertia
-      m="${mass_shoulder}"
+      m="${mass_elbow}"
       x="0.12"
       y="0.04"
@@ -121,5 +143,12 @@
   <child link="shoulder_link"/>
   <origin xyz="0 0.12124 0.06" rpy="0 0 0"/>
-  <axis xyz="0 1 0"/>
+  <axis xyz="0 0 1"/>
+  <limit lower="${-pi/2}" upper="${pi/2}" effort="50" velocity="1.0"/>
+</joint>
+<joint name="elbow_to_shoulder" type="revolute">
+  <parent link="shoulder_link"/>
+  <child link="elbow_link"/>
+  <origin xyz="0 0.358 0" rpy="0 0 0"/>
+  <axis xyz="0 0 1"/>
   <limit lower="${-pi/2}" upper="${pi/2}" effort="50" velocity="1.0"/>
 </joint>

Commit message: add new link

File: robot_description/urdf/scara_arm.xacro (robot description, xacro)
@@ -120,4 +120,26 @@
       o_rpy="0 0 0"/>
 </link>
+<link name="wrist_link">
+  <visual>
+    <geometry>
+      <mesh filename="file:///home/linos/cad_projects/gripper/v1.2/wrist.stl" scale="0.001 0.001 0.001"/>
+    </geometry>
+    <origin xyz="0 0.639 0.17" rpy="${pi} 0 0"/>
+    <material name="purple"/>
+  </visual>
+  <collision>
+    <geometry>
+      <box size="0.055 0.06 0.04"/>
+    </geometry>
+    <origin xyz="0 0 0" rpy="0 0 0"/>
+  </collision>
+  <xacro:box_inertia
+      m="${mass_wrist}"
+      x="0.055"
+      y="0.06"
+      z="0.04"
+      o_xyz="0 0 0"
+      o_rpy="0 0 0"/>
+</link>
 <joint name="arm_base_to_mobile_base_link" type="fixed">
   <parent link="mobile_uvc_base_link"/>
@@ -153,3 +175,10 @@
   <limit lower="${-pi/2}" upper="${pi/2}" effort="50" velocity="1.0"/>
 </joint>
+<joint name="elbow_to_wrist" type="revolute">
+  <parent link="elbow_link"/>
+  <child link="wrist_link"/>
+  <origin xyz="0 0.16 -0.42" rpy="0 ${pi} 0"/>
+  <axis xyz="0 0 1"/>
+  <limit lower="${-pi/2}" upper="${pi/2}" effort="50" velocity="1.0"/>
+</joint>
 </robot>
