Commit message: initialize arm modules in xacro

File: robot_description/urdf/arm.xacro (robot description, xacro)
@@ -1,3 +1,79 @@
 <?xml version="1.0"?>
 <robot xmlns:xacro="http://www.ros.org/wiki/xacro">
+<xacro:property name="arm_base_length" value="0.1"/>
+<xacro:property name="arm_base_width" value="0.1"/>
+<xacro:property name="arm_base_height" value="0.02"/>
+<xacro:property name="arm_length" value="0.3"/>
+<xacro:property name="arm_radius" value="0.02"/>
+<!-- Links -->
+<link name="arm_base_link">
+    <visual>
+        <geometry>
+            <box size="${arm_base_length} ${arm_base_width} ${arm_base_height}"/>
+        </geometry>
+        <origin xyz="0 0 0" rpy="0 0 0"/>
+        <material name="orange"/>
+    </visual>
+    <collision>
+        <geometry>
+            <box size="${arm_base_length} ${arm_base_width} ${arm_base_height}"/>
+        </geometry>
+        <origin xyz="0 0 0" rpy="0 0 0"/>
+    </collision>
+    <xacro:box_inertia m="0.5" x="${arm_base_length}" y="${arm_base_width}" z="${arm_base_height}" o_xyz="0 0 0" o_rpy="0 0 0"/>
+</link>
+<link name="forearm_link">
+    <visual>
+        <geometry>
+            <cylinder radius="${arm_radius}" length="${arm_length}"/>
+        </geometry>
+        <origin xyz="0 0 0" rpy="0 0 0"/>
+        <material name="yellow"/>
+    </visual>
+    <collision>
+        <geometry>
+            <cylinder radius="${arm_radius}" length="${arm_length}"/>
+        </geometry>
+        <origin xyz="0 0 0" rpy="0 0 0"/>
+    </collision>
+    <xacro:cylinder_inertia m="0.3" r="${arm_radius}" h="${arm_length}" o_xyz="0 0 0" o_rpy="0 0 0"/>
+</link>
+<link name="hand_link">
+    <visual>
+        <geometry>
+            <cylinder radius="${arm_radius}" length="${arm_length}"/>
+        </geometry>
+        <origin xyz="0 0 0" rpy="0 0 0"/>
+        <material name="orange"/>
+    </visual>
+    <collision>
+        <geometry>
+            <cylinder radius="${arm_radius}" length="${arm_length}"/>
+        </geometry>
+        <origin xyz="0 0 0" rpy="0 0 0"/>
+    </collision>
+    <xacro:cylinder_inertia m="0.3" r="${arm_radius}" h="${arm_length}" o_xyz="0 0 0" o_rpy="0 0 0"/>
+</link>
+<!-- Joints -->
+<joint name="arm_base_joint" type="fixed">
+    <parent link="mobile_base_link"/>
+    <child link="arm_base_link"/>
+    <origin xyz="0 0 0" rpy="0 0 0"/>
+</joint>
+<joint name="forearm_joint_to_arm_base" type="revolute">
+    <parent link="arm_base_link"/>
+    <child link="forearm_link"/>
+    <origin xyz="0 0 0" rpy="0 0 0"/>
+    <axis xyz="0 1 0"/>
+    <limit lower="0" upper="${pi/2}" effort="100" velocity="100"/>
+    <dynamics damping="0.3" friction="0.3"/>
+</joint>
+<joint name="hand_joint_to_forearm" type="revolute">
+    <parent link="forearm_link"/>
+    <child link="hand_link"/>
+    <origin xyz="0 0 0" rpy="0 0 0"/>
+    <axis xyz="0 1 0"/>
+    <limit lower="0" upper="${pi/2}" effort="100" velocity="100"/>
+    <dynamics damping="0.3" friction="0.3"/>
+</joint>
 </robot>

Commit message: update visual and joint axis

File: robot_description/urdf/arm.xacro (robot description, xacro)
@@ -28,5 +28,5 @@
             <cylinder radius="${arm_radius}" length="${arm_length}"/>
         </geometry>
-        <origin xyz="0 0 0" rpy="0 0 0"/>
+        <origin xyz="0 0 ${arm_length/2 - arm_base_height/2}" rpy="0 0 0"/>
         <material name="yellow"/>
     </visual>
@@ -35,7 +35,7 @@
             <cylinder radius="${arm_radius}" length="${arm_length}"/>
         </geometry>
-        <origin xyz="0 0 0" rpy="0 0 0"/>
+        <origin xyz="0 0 ${arm_length/2 - arm_base_height/2}" rpy="0 0 0"/>
     </collision>
-    <xacro:cylinder_inertia m="0.3" r="${arm_radius}" h="${arm_length}" o_xyz="0 0 0" o_rpy="0 0 0"/>
+    <xacro:cylinder_inertia m="0.3" r="${arm_radius}" h="${arm_length}" o_xyz="0 0 ${arm_length/2 - arm_base_height/2}" o_rpy="0 0 0"/>
 </link>
 <link name="hand_link">
@@ -44,5 +44,5 @@
             <cylinder radius="${arm_radius}" length="${arm_length}"/>
         </geometry>
-        <origin xyz="0 0 0" rpy="0 0 0"/>
+        <origin xyz="0 0 ${arm_length/2 - arm_base_height/2}" rpy="0 0 0"/>
         <material name="orange"/>
     </visual>
@@ -51,7 +51,7 @@
             <cylinder radius="${arm_radius}" length="${arm_length}"/>
         </geometry>
-        <origin xyz="0 0 0" rpy="0 0 0"/>
+        <origin xyz="0 0 ${arm_length/2 - arm_base_height/2}" rpy="0 0 0"/>
     </collision>
-    <xacro:cylinder_inertia m="0.3" r="${arm_radius}" h="${arm_length}" o_xyz="0 0 0" o_rpy="0 0 0"/>
+    <xacro:cylinder_inertia m="0.3" r="${arm_radius}" h="${arm_length}" o_xyz="0 0 ${arm_length/2 - arm_base_height/2}" o_rpy="0 0 0"/>
 </link>
 <!-- Joints -->
@@ -59,10 +59,10 @@
     <parent link="mobile_base_link"/>
     <child link="arm_base_link"/>
-    <origin xyz="0 0 0" rpy="0 0 0"/>
+    <origin xyz="${base_length/4} 0 ${arm_base_height/2 + base_height/2}" rpy="0 0 0"/>
 </joint>
 <joint name="forearm_joint_to_arm_base" type="revolute">
     <parent link="arm_base_link"/>
     <child link="forearm_link"/>
-    <origin xyz="0 0 0" rpy="0 0 0"/>
+    <origin xyz="0 0 ${arm_base_height}" rpy="0 0 0"/>
     <axis xyz="0 1 0"/>
     <limit lower="0" upper="${pi/2}" effort="100" velocity="100"/>
@@ -72,5 +72,5 @@
     <parent link="forearm_link"/>
     <child link="hand_link"/>
-    <origin xyz="0 0 0" rpy="0 0 0"/>
+    <origin xyz="0 0 ${arm_length}" rpy="0 0 0"/>
     <axis xyz="0 1 0"/>
     <limit lower="0" upper="${pi/2}" effort="100" velocity="100"/>

Commit message: code updates

File: robot_description/urdf/arm.xacro (robot description, xacro)
@@ -1,4 +1,2 @@
-<?xml version="1.0"?>
-<robot xmlns:xacro="http://www.ros.org/wiki/xacro">
 <xacro:property name="arm_base_length" value="0.1"/>
 <xacro:property name="arm_base_width" value="0.1"/>
@@ -77,3 +75,2 @@
     <dynamics damping="0.3" friction="0.3"/>
 </joint>
-</robot>

File: robot_description/urdf/camera.xacro (robot description, xacro)
@@ -20,5 +20,5 @@
     </link>
     <joint name="base_camera_joint" type="fixed">
-        <parent link="mobile_base_link" />
+        <parent link="mobile_uvc_base_link" />
         <child link="camera_link" />
         <origin xyz="${(base_length + camera_length) / 2.0} 0 ${base_height / 2.0}" rpy="0 0 0" />

File: robot_description/urdf/common_properties.xacro (robot description, xacro)
@@ -9,4 +9,5 @@
     <material name="red"><color rgba="1 0 0 1"/></material>
     <material name="gray"><color rgba="0.5 0.5 0.5 1"/></material>
+    <material name="grey"><color rgba="0.5 0.5 0.5 1"/></material>
     <!-- Common inertia calculations -->
     <xacro:macro name="box_inertia" params="m x y z o_xyz o_rpy">

File: robot_description/urdf/mobile_base.xacro (robot description, xacro)
@@ -1,4 +1,2 @@
-<?xml version="1.0"?>
-<robot xmlns:xacro="http://www.ros.org/wiki/xacro">
 <!-- Define mobile base properties -->
 <xacro:property name="base_length" value="0.6"/>
@@ -85,3 +83,2 @@
     <origin xyz="${base_length/4} 0 ${-(caster_radius+base_height/2)}" rpy="0 0 0"/>
 </joint>
-</robot>

File: robot_description/urdf/mobile_gazebo.xacro (robot description, xacro)
@@ -1,5 +1,5 @@
 <?xml version="1.0"?>
 <robot xmlns:xacro="http://www.ros.org/wiki/xacro">
-<gazebo reference="caster_wheel_link">
+<gazebo reference="roda_link">
     <mu1 value="0.1"/>
     <mu2 value="0.1"/>
@@ -11,5 +11,5 @@
         <left_joint>left_wheel_joint</left_joint>
         <right_joint>right_wheel_joint</right_joint>
-        <wheel_separation>${base_width + 2*wheel_width/2}</wheel_separation>
+        <wheel_separation>${base_width + wheel_width}</wheel_separation>
         <wheel_radius>${wheel_radius}</wheel_radius>
         <frame_id>odom</frame_id>
@@ -24,6 +24,12 @@
         <joint_name>left_wheel_joint</joint_name>
         <joint_name>right_wheel_joint</joint_name>
-        <joint_name>forearm_joint_to_arm_base</joint_name>
-        <joint_name>hand_joint_to_forearm</joint_name>
+        <joint_name>roda_joint</joint_name>
+        <joint_name>arm_base_to_waist</joint_name>
+        <joint_name>slide_carriage_to_slider</joint_name>
+        <joint_name>shoulder_to_slide_carriage</joint_name>
+        <joint_name>elbow_to_shoulder</joint_name>
+        <joint_name>wrist_to_elbow</joint_name>
+        <joint_name>left_finger_to_wrist</joint_name>
+        <joint_name>right_finger_to_wrist</joint_name>
     </plugin>
 </gazebo>

File: robot_description/urdf/mobile_manipulator.urdf.xacro (robot description, xacro)
@@ -4,7 +4,7 @@
 <xacro:include filename="common_properties.xacro"/>
 <!-- Include mobile base -->
-<xacro:include filename="mobile_base.xacro"/>
+<xacro:include filename="mobile_uvc.xacro"/>
 <!-- Include arm -->
-<xacro:include filename="arm.xacro"/>
+<xacro:include filename="scara_arm.xacro"/>
 <!-- Include mobile base gazebo plugins -->
  <xacro:include filename="mobile_gazebo.xacro" />

File: robot_description/urdf/mobile_uvc.xacro (robot description, xacro)
@@ -6,4 +6,7 @@
   <xacro:property name="wheel_radius" value="0.119289"/>
   <xacro:property name="wheel_width" value="0.160767"/>
+  <xacro:property name="base_width" value="0.478531"/>
+  <xacro:property name="base_length" value="0.849993"/>
+  <xacro:property name="base_height" value="0.253914"/>
   <xacro:property name="roda_radius" value="0.038463"/>
   <xacro:property name="base_x" value="0.102772"/>

File: robot_description/urdf/scara_arm.xacro (robot description, xacro)
@@ -15,5 +15,5 @@
   <visual>
     <geometry>
-      <mesh filename="file:///home/linos/cad_projects/gripper/v1.2/base.stl" scale="0.001 0.001 0.001"/>
+      <mesh filename="file:///home/linos/cad_projects/gripper/base.stl" scale="0.001 0.001 0.001"/>
     </geometry>
     <origin xyz="0 0 0" rpy="0 0 0"/>
@@ -35,5 +35,5 @@
   <visual>
     <geometry>
-      <mesh filename="file:///home/linos/cad_projects/gripper/v1.2/waist.stl" scale="0.001 0.001 0.001"/>
+      <mesh filename="file:///home/linos/cad_projects/gripper/waist.stl" scale="0.001 0.001 0.001"/>
     </geometry>
     <origin xyz="0 0 ${-base_cylinder_height}" rpy="0 0 0"/>
@@ -57,5 +57,5 @@
   <visual>
     <geometry>
-      <mesh filename="file:///home/linos/cad_projects/gripper/v1.2/slider_carriage.stl" scale="0.001 0.001 0.001"/>
+      <mesh filename="file:///home/linos/cad_projects/gripper/slider_carriage.stl" scale="0.001 0.001 0.001"/>
     </geometry>
     <origin xyz="0 0 ${-slider_length - base_cylinder_height}" rpy="0 0 0"/>
@@ -79,5 +79,5 @@
   <visual>
     <geometry>
-      <mesh filename="file:///home/linos/cad_projects/gripper/v1.2/shoulder.stl" scale="0.001 0.001 0.001"/>
+      <mesh filename="file:///home/linos/cad_projects/gripper/shoulder.stl" scale="0.001 0.001 0.001"/>
     </geometry>
     <origin xyz="0 -0.1212 ${-slider_length + base_cylinder_height - 2 * 0.09}" rpy="0 0 0"/>
@@ -101,5 +101,5 @@
   <visual>
     <geometry>
-      <mesh filename="file:///home/linos/cad_projects/gripper/v1.2/elbow.stl" scale="0.001 0.001 0.001"/>
+      <mesh filename="file:///home/linos/cad_projects/gripper/elbow.stl" scale="0.001 0.001 0.001"/>
     </geometry>
     <origin xyz="0 ${-0.48} ${-slider_length + base_cylinder_height - 2 * 0.09}" rpy="0 0 0"/>
@@ -123,5 +123,5 @@
   <visual>
     <geometry>
-      <mesh filename="file:///home/linos/cad_projects/gripper/v1.2/wrist.stl" scale="0.001 0.001 0.001"/>
+      <mesh filename="file:///home/linos/cad_projects/gripper/wrist.stl" scale="0.001 0.001 0.001"/>
     </geometry>
     <origin xyz="0 0.639 0.17" rpy="${pi} 0 0"/>
@@ -145,5 +145,5 @@
   <visual>
     <geometry>
-      <mesh filename="file:///home/linos/cad_projects/gripper/v1.2/left_finger.stl" scale="0.001 0.001 0.001"/>
+      <mesh filename="file:///home/linos/cad_projects/gripper/left_finger.stl" scale="0.001 0.001 0.001"/>
     </geometry>
     <origin xyz="-0.02 -0.639 0.06" rpy="0 ${pi} 0"/>
@@ -167,5 +167,5 @@
   <visual>
     <geometry>
-      <mesh filename="file:///home/linos/cad_projects/gripper/v1.2/right_finger.stl" scale="0.001 0.001 0.001"/>
+      <mesh filename="file:///home/linos/cad_projects/gripper/right_finger.stl" scale="0.001 0.001 0.001"/>
     </geometry>
     <origin xyz="0.02 -0.639 0.06" rpy="0 ${pi} 0"/>
